File: hardware/development/Kampela_C1/display.kicad_sch (KiCad schematic)
At the start: 39 parts, among them Q3 SSM6N35AFE

Commit message: feat: initial routing
Parts:
- added C?: 4.7x25, Capacitor_SMD:C_0402_1005Metric, symbol Device:C
- J?: footprint 123123:GDEY0154D67_TP_bended -> MyLib:GDEY027T91-T01_bended
- J?: footprint 123123:HRS_FH34SRJ-6S-0.5SH(50) -> MyLib:HRS_FH34SRJ-6S-0.5SH(50)
- U?: footprint Package_DFN_QFN:Texas_R_PUQFN-N12 -> Package_DFN_QFN:Texas_R-PUQFN-N12
Connections:
- net +2V8: now also C?.2, J?.15 (Pin_15), J?.16 (Pin_16), J?.4 (Pin_4), C?.1
- net GND: now also C?.2
- net POW: no longer C?.2, J?.15 (Pin_15), J?.16 (Pin_16), J?.4 (Pin_4)
Other:
- moved on the sheet: C?
Changed lines of the file:
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@@
 (kicad_sch (version 20221206) (generator eeschema)
   (paper "A4")
+  (junction (at 234.95 49.53) (diameter 0) (color 0 0 0 0)
+  )
   (junction (at 168.91 74.93) (diameter 0) (color 0 0 0 0)
   )
@@
     (stroke (width 0) (type default))
   )
+  (wire (pts (xy 83.82 86.36) (xy 83.82 87.63))
+    (stroke (width 0) (type default))
+  )
   (wire (pts (xy 114.3 74.93) (xy 114.3 77.47))
     (stroke (width 0) (type default))
@@
     (stroke (width 0) (type default))
   )
+  (wire (pts (xy 228.6 49.53) (xy 234.95 49.53))
+    (stroke (width 0) (type default))
+  )
   (wire (pts (xy 191.77 62.23) (xy 205.74 62.23))
     (stroke (width 0) (type default))
@@
     (stroke (width 0) (type default))
   )
-  (wire (pts (xy 83.82 74.93) (xy 83.82 80.01))
+  (wire (pts (xy 83.82 74.93) (xy 83.82 78.74))
     (stroke (width 0) (type default))
   )
@@
     (stroke (width 0) (type default))
   )
-  (wire (pts (xy 233.68 41.91) (xy 242.57 41.91))
+  (wire (pts (xy 228.6 41.91) (xy 242.57 41.91))
     (stroke (width 0) (type default))
   )
@@
     (stroke (width 0) (type default))
   )
-  (wire (pts (xy 93.98 80.01) (xy 93.98 74.93))
+  (wire (pts (xy 93.98 78.74) (xy 93.98 74.93))
     (stroke (width 0) (type default))
   )
@@
     (stroke (width 0) (type default))
   )
+  (wire (pts (xy 93.98 86.36) (xy 93.98 87.63))
+    (stroke (width 0) (type default))
+  )
   (wire (pts (xy 191.77 57.15) (xy 205.74 57.15))
     (stroke (width 0) (type default))
@@
     (effects (font (size 1.27 1.27)) (justify left bottom))
   )
+  (label "+2V8" (at 189.23 74.93 0) (fields_autoplaced)
+    (effects (font (size 1.27 1.27)) (justify left bottom))
+  )
   (label "VCOM" (at 191.77 95.25 0) (fields_autoplaced)
     (effects (font (size 1.27 1.27)) (justify left bottom))
   )
-  (label "POW" (at 233.68 41.91 0) (fields_autoplaced)
+  (label "+2V8" (at 233.68 41.91 0) (fields_autoplaced)
     (effects (font (size 1.27 1.27)) (justify left bottom))
   )
@@
   )
   (label "T_SDA" (at 198.12 107.95 0) (fields_autoplaced)
-    (effects (font (size 1.27 1.27)) (justify left bottom))
-  )
-  (label "POW" (at 191.77 74.93 0) (fields_autoplaced)
     (effects (font (size 1.27 1.27)) (justify left bottom))
   )
@@
     )
   )
-  (symbol (lib_id "Device:C") (at 93.98 83.82 0) (unit 1)
-    (in_bom yes) (on_board yes) (dnp no)
-    (property "Reference" "C?" (at 87.63 85.09 0)
-      (effects (font (size 1.27 1.27)) (justify left))
-    )
-    (property "Value" "0.1" (at 87.63 82.55 0)
-      (effects (font (size 1.27 1.27)) (justify left))
-    )
-    (property "Footprint" "Capacitor_SMD:C_0402_1005Metric" (at 94.9452 87.63 0)
-      (effects (font (size 1.27 1.27)) hide)
-    )
-    (property "Datasheet" "~" (at 93.98 83.82 0)
+  (symbol (lib_id "Device:C") (at 93.98 82.55 0) (unit 1)
+    (in_bom yes) (on_board yes) (dnp no)
+    (property "Reference" "C?" (at 87.63 83.82 0)
+      (effects (font (size 1.27 1.27)) (justify left))
+    )
+    (property "Value" "0.1" (at 87.63 81.28 0)
+      (effects (font (size 1.27 1.27)) (justify left))
+    )
+    (property "Footprint" "Capacitor_SMD:C_0402_1005Metric" (at 94.9452 86.36 0)
+      (effects (font (size 1.27 1.27)) hide)
+    )
+    (property "Datasheet" "~" (at 93.98 82.55 0)
       (effects (font (size 1.27 1.27)) hide)
     )
@@
       (effects (font (size 1.27 1.27)) (justify left))
     )
-    (property "Footprint" "Package_DFN_QFN:Texas_R_PUQFN-N12" (at 52.07 147.32 0)
+    (property "Footprint" "Package_DFN_QFN:Texas_R-PUQFN-N12" (at 52.07 147.32 0)
       (effects (font (size 1.27 1.27)) hide)
     )
@@
     )
   )
+  (symbol (lib_id "Device:C") (at 228.6 45.72 0) (unit 1)
+    (in_bom yes) (on_board yes) (dnp no)
+    (property "Reference" "C?" (at 219.71 40.64 0)
+      (effects (font (size 1.27 1.27)) (justify left))
+    )
+    (property "Value" "4.7x25" (at 219.71 43.18 0)
+      (effects (font (size 1.27 1.27)) (justify left))
+    )
+    (property "Footprint" "Capacitor_SMD:C_0402_1005Metric" (at 229.5652 49.53 0)
+      (effects (font (size 1.27 1.27)) hide)
+    )
+    (property "Datasheet" "~" (at 228.6 45.72 0)
+      (effects (font (size 1.27 1.27)) hide)
+    )
+    (pin "1")
+    (pin "2")
+    (instances
+      (project "Kampela"
+        (path "/472e0f49-51e5-4b9c-a9f6-6aed0741c677/7868ecaa-9431-43d7-95a8-9c0f01ec9958"
+          (reference "C?") (unit 1)
+        )
+      )
+      (project "Kampela_C1"
+        (path "/f1094595-086c-43ea-a0be-6f801d9d8744/7868ecaa-9431-43d7-95a8-9c0f01ec9958"
+          (reference "C57") (unit 1)
+        )
+      )
+    )
+  )
   (symbol (lib_id "Connector_Generic:Conn_01x24") (at 210.82 64.77 0) (unit 1)
     (in_bom yes) (on_board yes) (dnp no)
@@
       (effects (font (size 1.27 1.27)))
     )
-    (property "Footprint" "123123:GDEY0154D67_TP_bended" (at 210.82 64.77 0)
+    (property "Footprint" "MyLib:GDEY027T91-T01_bended" (at 210.82 64.77 0)
       (effects (font (size 1.27 1.27)) hide)
     )
@@
       (effects (font (size 1.27 1.27)))
     )
-    (property "Footprint" "123123:HRS_FH34SRJ-6S-0.5SH(50)" (at 247.65 44.45 0)
+    (property "Footprint" "MyLib:HRS_FH34SRJ-6S-0.5SH(50)" (at 247.65 44.45 0)
       (effects (font (size 1.27 1.27)) hide)
     )
@@
     )
   )
-  (symbol (lib_id "Device:C") (at 83.82 83.82 180) (unit 1)
-    (in_bom yes) (on_board yes) (dnp no)
-    (property "Reference" "C?" (at 80.01 85.09 0)
-      (effects (font (size 1.27 1.27)) (justify left))
-    )
-    (property "Value" "4.7x25" (at 80.01 82.55 0)
-      (effects (font (size 1.27 1.27)) (justify left))
-    )
-    (property "Footprint" "Capacitor_SMD:C_0402_1005Metric" (at 82.8548 80.01 0)
-      (effects (font (size 1.27 1.27)) hide)
-    )
-    (property "Datasheet" "~" (at 83.82 83.82 0)
-      (effects (font (size 1.27 1.27)) hide)
-    )
+  (symbol (lib_id "Device:C") (at 83.82 82.55 180) (unit 1)
+    (in_bom yes) (on_board yes) (dnp no)
+    (property "Reference" "C?" (at 80.01 83.82 0)
+      (effects (font (size 1.27 1.27)) (justify left))
+    )
+    (property "Value" "4.7x25" (at 80.01 81.28 0)
+      (effects (font (size 1.27 1.27)) (justify left))
+    )
+    (property "Footprint" "Capacitor_SMD:C_0402_1005Metric" (at 82.8548 78.74 0)
+      (effects (font (size 1.27 1.27)) hide)
+    )
+    (property "Datasheet" "~" (at 83.82 82.55 0)
+      (effects (font (size 1.27 1.27)) hide)
+    )
