File: hardware/development/Kampela_C1/mcu.kicad_sch (KiCad schematic)
At the start: 20 parts, among them J3 SOICbite, U5 AT25XE321D-UUN-T, U6 EFM32PG23B200F512IM40, Y2 39MHz

Commit message: feat: initial routing
Parts:
- added J6: Conn_01x08, Connector_PinHeader_1.00mm:PinHeader_1x08_P1.00mm_Vertical, symbol Connector_Generic:Conn_01x08
- D8: footprint Package_TO_SOT_SMD:SOT-523 -> MyLib:SOT-523
- U?: footprint 123123:SON-8-1EP_3x2mm_P0.5mm_EP1.4x1.6mm -> MyLib:SON-8-1EP_3x2mm_P0.5mm_EP1.4x1.6mm
- Y?: footprint 123123:Crystal_SMD_2012-2Pin_2.0x1.2mm -> MyLib:Crystal_SMD_2012-2Pin_2.0x1.2mm
Connections:
- net +1V8: now also J6.1 (Pin_1)
- net BUSY: now also U6.15 (PB04); no longer U6.25 (PA05)
- net CS: now also U6.38 (PD02); no longer U6.18 (PB01)
- net DATA: now also U6.28 (PA08); no longer U6.19 (PB00)
- net D/C: now also U6.37 (PD03); no longer U6.27 (PA07)
- net E_MISO: now also U6.2 (PC01); no longer U6.4 (PC03)
- net GND: now also J6.4 (Pin_4)
- net I2C_P: now also U6.24 (PA04); no longer U6.23 (PA03)
- net INT: now also U6.18 (PB01); no longer U6.15 (PB04)
- net P_GOOD: now also J6.8 (Pin_8)
- net RX: now also U6.14 (PB05), J6.2 (Pin_2); no longer U6.13 (PB06)
- net R_MISO: now also U6.6 (PC05); no longer U6.8 (PC07)
- net R_SCK: now also U6.8 (PC07); no longer U6.6 (PC05)
- net SCK: now also U6.4 (PC03); no longer U6.2 (PC01)
- net SCL: now also U6.23 (PA03); no longer U6.16 (PB03)
- net SDA: now also U6.25 (PA05); no longer U6.17 (PB02)
- net SWDCK: now also J6.7 (Pin_7)
- net SWDIO: now also J6.5 (Pin_5)
- net TX: now also U6.13 (PB06), J6.3 (Pin_3); no longer U6.14 (PB05)
- net P_IN: now reaches D?.2 (A), J3.6 (Pin_6), R?.1
- net P_IN: now also J6.6 (Pin_6)
- no-connect marks 9 -> 7
Other:
- moved on the sheet: C?, Y?
