File: hardware/development/Kampela_C1/power.kicad_sch (KiCad schematic)
At the start: 54 parts

Commit message: feat: initial routing
Parts:
- added C? (x29): 47x16, Capacitor_SMD:C_1210_3225Metric, symbol Device:C
- J? (x2): footprint 123123:TestPoint_Pad_2.4x3.5mm -> MyLib:TestPoint_Pad_2.4x3.5mm
- JP?: footprint 123123:SolderJumper_0.8.x1mm -> MyLib:SolderJumper_0.8.x1mm
Connections:
- net HV: now also C?.2, C?.2, C?.2, C?.2, C?.2, C?.2, C?.2, C?.2, C?.2, C?.2, C?.2, C?.2, C?.2, C?.2, C?.2, C?.2, C?.2, C?.2, C?.2, C?.2, C?.2, C?.2, C?.2, C?.2, C?.2, C?.2, C?.2, C?.2, C?.2
- net CN: now reaches C?.1, C?.1, C?.1, C?.1, C?.1, C?.1, C?.1, C?.1, JP?.2 (B), Q?.3 (D)
- net CN: now also C?.1, C?.1, C?.1, C?.1, C?.1, C?.1, C?.1, C?.1, C?.1, C?.1, C?.1, C?.1, C?.1, C?.1, C?.1, C?.1, C?.1, C?.1, C?.1, C?.1, C?.1, C?.1, C?.1, C?.1, C?.1, C?.1, C?.1, C?.1, C?.1
