File: hardware/development/Kampela_C1/Kampela_C1.kicad_pcb (KiCad board)
At the start: 2 copper layers, 115 x 46 mm, 163 parts, among them J1 E_ANT, J2 E_ANT, J3 SOICbite, J4 E2154CS0C1, J5 TOUCH, J6 Conn_01x08, Q1 PMF250XNEX, Q2 PMF250XNEX, Q3 SSM6N35AFE, Q4 2N7002KW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

Commit message: feat: pcb labels
Parts:
- added G***: LOGO, LOGO, B.Cu at (84.3, 119.1)
- moved D3 8.47 mm to (139.5, 128.8)
- moved JP3 4.76 mm to (138.5, 103.1), turned to -90 degrees
- moved R7 4.51 mm to (137.5, 132.2), turned to -90 degrees
- turned C58 to 90 degrees
- turned C59 to 90 degrees
- turned C60 to 90 degrees
- turned C61 to 90 degrees
- turned C62 to 90 degrees
- turned C63 to 90 degrees
- turned C64 to 90 degrees
- turned C65 to 90 degrees
- turned C66 to 90 degrees
- turned C67 to 90 degrees
- turned C68 to 90 degrees
- turned C69 to 90 degrees
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- renumbered TP2 to 1V8, TP3 to 2V8, TP1 to DT, TP6 to VC, TP5 to VGH, TP4 to VGL
Routing:
- net /MCU/HV: track 273.0 -> 271.2 mm
- net Net-(D3-A): track 4.74 -> 3.59 mm
- net /Power/CN: track 187.8 -> 187.6 mm, vias 4 -> 2
- net GND: vias 518 -> 525
Other:
- board text added: "+"
- board text added: "2023"
- board text added: "C"
- board text added: "RST DCK POW DIO GND TX RX 1V8"

Commit message: feat: update C1 version; add D version and tag
Parts:
- added JP3: SolderJumper_2_Open, MyLib:SolderJumper_0.8.x1mm, F.Cu at (141.0, 109.7)
- added JP3: SolderJumper_2_Open, MyLib:SolderJumper_0.8.x1mm, F.Cu at (141.0, 115.2)
- added JP3: SolderJumper_2_Open, MyLib:SolderJumper_0.8.x1mm, F.Cu at (141.0, 131.7)
- added JP3: SolderJumper_2_Open, MyLib:SolderJumper_0.8.x1mm, F.Cu at (141.0, 137.2)
- added JP3: SolderJumper_2_Open, MyLib:SolderJumper_0.8.x1mm, F.Cu at (141.0, 120.7)
- added JP3: SolderJumper_2_Open, MyLib:SolderJumper_0.8.x1mm, F.Cu at (141.0, 126.2)
- added JP3: SolderJumper_2_Open, MyLib:SolderJumper_0.8.x1mm, F.Cu at (141.0, 104.2)
- renumbered DT to TP1, 1V8 to TP2, 2V8 to TP3, VGL to TP4, VGH to TP5, VC to TP6
Routing:
- net /Power/CN: track 187.6 -> 170.8 mm
- net GND: vias 525 -> 537
