File: hardware/development/Kampela_D/rxfilter.kicad_sch (KiCad schematic)
At the start: 23 parts

Commit message: feat: update C1 version; add D version and tag
Parts:
- removed C?: 100p, Capacitor_SMD:C_0402_1005Metric, symbol Device:C
- removed C? (x2): 0.1u, Capacitor_SMD:C_0402_1005Metric, symbol Device:C
- removed FB?: BLM15AG102SZ1D, Inductor_SMD:L_0402_1005Metric, symbol Device:FerriteBead_Small
- removed R?: 47K, Resistor_SMD:R_0402_1005Metric, symbol Device:R
- removed R?: 22K, Resistor_SMD:R_0402_1005Metric, symbol Device:R
- removed R?: 10K, Resistor_SMD:R_0402_1005Metric, symbol Device:R
- removed R?: 100K, Resistor_SMD:R_0402_1005Metric, symbol Device:R
- removed U?: LMV7271, Package_TO_SOT_SMD:SOT-353_SC-70-5, symbol Comparator:LMV7271
- C?: value 100p -> 82p
- C?: value 47p -> 100p
- R?: value 10K -> 47K
- R?: value 10K -> 6.8K
- R?: value 51K -> 100K
Other:
- note removed: "100p"
- note removed: "6.8K"
- note removed: "82p"
- moved on the sheet: C?
