File: hardware/development/Kampela_D/display.kicad_sch (KiCad schematic)
At the start: 40 parts, among them Q3 SSM6N35AFE

Commit message: major: first device prototype (#24)
* feat: initial routing

* feat: pcb labels

* feat: update C1 version; add D version and tag
Parts:
- removed Q?: 2N7002KW, Package_TO_SOT_SMD:SOT-323_SC-70, symbol Device:Q_NMOS_GSD
- added Q4: SSM6N35AFE, Package_TO_SOT_SMD:SOT-563, symbol Transistor_FET:FDG1024NZ
- added R? (x2): 10K, Resistor_SMD:R_0402_1005Metric, symbol Device:R
- added R?: 100, Resistor_SMD:R_0402_1005Metric, symbol Device:R
- added R?: 1K, Resistor_SMD:R_0402_1005Metric, symbol Device:R
Connections:
- net +2V8: now also R?.2
- net E_RES: now also Q4.6 (D); no longer J?.3 (Pin_3)
- net GND: now also J?.S2 (S), J?.S2 (S), Q4.1 (S), Q4.3 (D), R?.1
- net H_SDI: now also R?.1, R?.2; no longer U?.10 (B1)
- net RES: now also Q4.2 (G)
- net I2C_P renamed 2V8_EN
- new net: R?.2, U?.10 (B1)
- new net E_MISO: R?.1
- new net RES_TC: Q4.5 (G), R?.2
- new net T_RES: J?.3 (Pin_3), Q4.4 (S), R?.1
Other:
- moved on the sheet: C?, D?, FB?, L?, Q3A, Q3B, Q?, R?, TP?, U?
