File: hardware/development/Kampela_D/mcu.kicad_sch (KiCad schematic)
At the start: 21 parts, among them J3 SOICbite, J6 Conn_01x08, U5 AT25XE321D-UUN-T, U6 EFM32PG23B200F512IM40, Y2 39MHz

Commit message: major: first device prototype (#24)
* feat: initial routing

* feat: pcb labels

* feat: update C1 version; add D version and tag
Parts:
- removed D8: BAT54CT, MyLib:SOT-523, symbol Diode:BAT54C
- added J7: Conn_01x02, Connector_PinHeader_1.27mm:PinHeader_1x02_P1.27mm_Vertical, symbol Connector_Generic:Conn_01x02
- added R?: 2.2, Resistor_SMD:R_0603_1608Metric, symbol Device:R
- added TP? (x2): TestPoint, TestPoint:TestPoint_Pad_D1.0mm, symbol Connector:TestPoint
- J6: footprint Connector_PinHeader_1.00mm:PinHeader_1x08_P1.00mm_Vertical -> Connector_PinHeader_1.27mm:PinHeader_1x08_P1.27mm_Vertical
Connections:
- net I2C_P is gone; now on net SCL: U6.24 (PA04)
- net DATA: now also TP?.1
- net P_IN: now also R?.1; no longer D?.2 (A), R?.1
- net SCL: no longer U6.23 (PA03)
- net at U6.16 (PB03): now also J7.2 (Pin_2)
- net at U6.17 (PB02): now also J7.1 (Pin_1)
- net at U6.19 (PB00): now also TP?.1
- net RES_TC: now reaches U6.27 (PA07)
- new net: D?.2 (A), R?.1, R?.2
- new net ~{MCU_OK}: U6.23 (PA03)
- no-connect marks 7 -> 5
Other:
- moved on the sheet: C?, D?, FB?, J3, J6, R?, U5, U6, U?, Y2, Y?
